File: Xenia1-MaGP-I-Electronics/Xenia1-MaGP-I-Electronics.kicad_sch (KiCad schematic)
At the start: 17 parts, among them Q1 Q_NPN_EBC, U1 BOOST_CONVERTER, U2 BMP_390, U3 ADAFRUIT_MPU_6050, U4 SD_CARD_READER, U5 HALL_EFFECT_SENSOR, U6 NEO-7M_GPS_MODULE, U7 L293D, U8 12V_DC_MOTOR+ENCODER, U9 TELEGPS

Commit message: Updated I/O Pin Assignment
Updated wiring diagram according to the actual wiring
Parts:
- removed Q1: Q_NPN_EBC, symbol Device:Q_NPN_EBC
- removed U4: SD_CARD_READER, symbol MaGP-I_Library:SD_CARD_READER
Connections:
- net A4 (SDA0): now also U3. (VIN)
- net A5 (SCL0): now also U3. (VIN)
- net GND: no longer BT2.2 (-)
- net D31: now reaches U?.31 (CTX3)
- net D31: now also U8.3 (C1)
- net D32: now reaches U?.32 (OUT1B)
- net D32: now also U8.4 (C2)
- net D34 (RX8): now reaches U?.34 (RX8)
- net D34 (RX8): now also U6. (VCC)
- net D35 (TX8): now reaches U?.35 (TX8)
- net D35 (TX8): now also U6. (VCC)
- net at U9. (GND1): now also BT2.2 (-)
- net D1: now reaches IC?.23 (GPIO_11/SPI0_SCLK)
- net D1: now also U?.1 (TX1)
- net A2 (SCL1): no longer names the net of U?.16 (A2)
- net A2 (SCL1): no longer U3. (VIN)
- net A3 (SDA1): no longer names the net of U?.17 (A3)
- net A3 (SDA1): no longer U3. (VIN)
- net D0 (RX1): no longer names the net of U?.0 (RX1)
- net D0 (RX1): no longer U6. (VCC)
- removed net D1 (TX1): U6. (VCC), U?.1 (TX1)
- net D2: no longer names the net of U?.2 (OUT2)
- net D20: no longer names the net of U?.20 (A6)
- net D20: no longer U8.4 (C2)
- net D21: no longer names the net of U?.21 (A7)
- net D21: no longer U8.3 (C1)
- net D22 renamed D12
- net D6: no longer names the net of U?.6 (OUT1D)
- net D6: no longer IC?.3 (GPIO_2/[I2C]_SDA)
Other:
- note added: "6-JUNE-2022"
- note added: "?"
- note added: "NOTE: 1. TELEGPS IS A STANDALONE UNIT IN MAGPI, THERE IS NO INTERNAL INTERACTION WITH OTHER COMPONENTS"
- note added: "SERIAL (UART)"
- note added: "TELEGPS*"
- note removed: "SPI DEVICES"
- moved on the sheet: BT2, U2, U3, U6, U9
